File: HW/AFE/AFE.sch (KiCad schematic (older format))
At the start: 49 parts

Commit message: updates
Parts:
- removed C?: 1000pF, symbol C_Small
- removed C?: 0.33uF, symbol C_Small
- added C? (x4): 0.33uF, symbol C_Small
- added C? (x9): 0.1uF, symbol C_Small
- added C?: 1000pF, symbol C_Small
- added C? (x7): 2.2uF, symbol C_Small
- added C? (x6): 1uF, symbol C_Small
- added C? (x3): 4.7uF, symbol C_Small
- added L?: 6.8uH, symbol L
- added R? (x8): R, symbol R
- added U?: ISA0505, symbol ISA0505
- added U? (x2): MAX8892, symbol MAX8892
- added U? (x2): MAX1735, symbol MAX1735
Connections:
- net labels added: -3V
- net labels removed: -5V
- wire segments 139 -> 253
Other:
- moved on the sheet: C?, J?, R?, T?, U?
